File: Board Files/Schematic.sch (KiCad schematic (older format))
At the start: 55 parts, among them P1-72EDGE1 CONN-NES-CARTRIDGE, P2-EXP1 SOCKET-50V, Q3 2SD1048-7-TB-E, Q4 2SD1048-7-TB-E, U1-WRAM1 DIL24-6, U10-CIC1 10NES, U2-LATCH1 SN74LS373DW, U3-DEMUX1 74139N, U4-VRAM1 DIL24-6, U5-PPU1 2C02, U6-CPU1 2A03, U7-HEXBUFFER1 CD74HC368M, U8-HEXBUFFER2 CD74HC368M, U9-HEXINVERTER1 SN74HC04N

Commit message: 
Parts:
- removed C1, C2, C3, C4, C5, C6, C7, C8: 330pF, NesRE:C0805, symbol NesRE-eagle-import:C-USC0805
- removed C10: 0.47u, NesRE:C050-035X075, symbol NesRE-eagle-import:C-US050-035X075
- removed C11, C12: 220pF, NesRE:C0402, symbol NesRE-eagle-import:C-USC0402
- removed C13, C14: 51pF, NesRE:C0603, symbol NesRE-eagle-import:C-USC0603
- removed C15, C16: 15pF, NesRE:C0603, symbol NesRE-eagle-import:C-USC0603
- removed C17: 30pF, NesRE:C0603, symbol NesRE-eagle-import:C-USC0603
- removed C18: C-USC0603, NesRE:C0603, symbol NesRE-eagle-import:C-USC0603
- removed DA1, DA2: 82401646, NesRE:SOP65P488X107-8N, symbol NesRE-eagle-import:82401646
- removed P1-72EDGE1: CONN-NES-CARTRIDGE, NesRE:CONN-NES-CARTRIDGE, symbol NesRE-eagle-import:CONN-NES-CARTRIDGE
- removed P2-EXP1: SOCKET-50V, NesRE:S50V, symbol NesRE-eagle-import:SOCKET-50V
- removed Q3, Q4: 2SD1048-7-TB-E, NesRE:SOT23, symbol NesRE-eagle-import:BC848SMD
- removed R1, R11, R12, R14, R15, R16, R17, R18, R19, R2, R3, R5: 10K, NesRE:M0805, symbol NesRE-eagle-import:R-US_M0805
- removed R10: 220K, NesRE:R0805, symbol NesRE-eagle-import:R-US_R0805
- removed R13, R4: 5600, NesRE:M0805, symbol NesRE-eagle-import:R-US_M0805
- removed R6: 1M, NesRE:R0402, symbol NesRE-eagle-import:R-US_R0402
- removed R7: 150K, NesRE:R0805, symbol NesRE-eagle-import:R-US_R0805
- removed R8, R9: 510, NesRE:R0805, symbol NesRE-eagle-import:R-US_R0805
- removed RST_SW1: MX1A-E1NW, NesRE:CHERRY-MX, symbol NesRE-eagle-import:CHERRY-MX
- removed U1-WRAM1, U4-VRAM1: DIL24-6, NesRE:DIL24-6, symbol NesRE-eagle-import:DIL24-6
- removed U10-CIC1: 10NES, NesRE:SOCKET-16, symbol NesRE-eagle-import:DIL16S
- removed U2-LATCH1: SN74LS373DW, NesRE:SOIC127P1030X265-20N, symbol NesRE-eagle-import:SN74LS373DW
- removed U3-DEMUX1: 74139N, NesRE:DIL16, symbol NesRE-eagle-import:74139N
- removed U5-PPU1: 2C02, NesRE:DIL40, symbol NesRE-eagle-import:2C02
- removed U6-CPU1: 2A03, NesRE:DIL40, symbol NesRE-eagle-import:2A03
- removed U7-HEXBUFFER1, U8-HEXBUFFER2: CD74HC368M, NesRE:SOIC127P600X175-16N, symbol NesRE-eagle-import:CD74HC367M
- removed U9-HEXINVERTER1: SN74HC04N, NesRE:DIP254P762X508-14, symbol NesRE-eagle-import:SN74HC04N
- removed XTAL3: 4Mhz, NesRE:HC49U, symbol NesRE-eagle-import:8M10AHC49T
- removed XTAL4: 21.47727 Mhz, NesRE:HC49U, symbol NesRE-eagle-import:8M10AHC49T
- added BC1, BC2: 103-25, Capacitor_THT:C_Disc_D6.0mm_W2.5mm_P5.00mm, symbol Device:C_Small
- added C1: 100uF, Capacitor_THT:CP_Radial_D5.0mm_P2.50mm, symbol Device:CP_Small
- added C10, C12, C13, C15, C16, C19, C2, C22, C24, C26, C3, C32, C38, C39, C40: 10nF, Capacitor_THT:C_Disc_D5.0mm_W2.5mm_P5.00mm, symbol Device:C_Small
- added C11, C14, C17, C18: 10nF, symbol Device:C_Small
- added C20, C43, C45: 51pF, symbol Device:C_Small
- added C21, C4, C44, C6, C7: 220pF, symbol Device:C_Small
- added C23: 1uF, symbol Device:CP_Small
- added C25: (Unused), Capacitor_THT:C_Disc_D5.0mm_W2.5mm_P5.00mm, symbol Device:C_Small
- added C27, C28, C29, C30, C31, C33, C34, C35, C36, C37: 330pF, Capacitor_THT:C_Disc_D3.0mm_W1.6mm_P2.50mm, symbol Device:C_Small
- added C41: 18pF, symbol Device:C_Small
- added C42: 15pF, symbol Device:C_Small
- added C46: 100nF, Capacitor_THT:C_Disc_D7.0mm_W2.5mm_P5.00mm, symbol Device:C_Small
- added C47, C48: (Unused), symbol Device:C_Small
- added C5: 330pF, symbol Device:C
- added C8: 100nF, symbol Device:C_Small
- added C9: 2.2uF, symbol Device:CP_Small
- added Controller_Port_1: Joystick_I, symbol NES-CPU-11:Controller_Port
- added Controller_Port_2: Joystick_II, symbol NES-CPU-11:Controller_Port
- added D1, D10, D11, D12, D13, D14, D2, D3, D4, D5, D6, D7, D8, D9: ?, symbol Device:D
- added DA1, DA3: DAN601, Resistor_THT:R_Array_SIP7, symbol Schematic:Diode_Array_7pin_(Cathode-Common)
- added DA2, DA4: UPA64H, Resistor_THT:R_Array_SIP7, symbol Schematic:Diode_Array_7pin_(Anode-Common)
- added FC1: 39u, symbol Schematic:Ferrite_Core
- added FC2: Ferrite_Coil, symbol Device:L_Core_Ferrite
- added J1, J2: Controller Output, symbol Connector:Conn_01x07_Male
- added LED1: POWERLED, symbol Device:LED
- added P1: 72-Pin Connector, symbol NES-CPU-11:72-Pin_Connector
- added P2: EXP-Connector, NesRE:NES_Edge_Connector, symbol NES-CPU-11:EXP-CON
- added P3: MOD RF, symbol Connector:Conn_01x05_Male
- added P4, P5: Controller Input, symbol Connector:Conn_01x07_Female
- added P6: PWR/RST IN, symbol Connector:Conn_01x05_Male
- added P7: PWR/RST OUT, symbol Connector:Conn_01x05_Female
- added Q1: 2SA937, symbol Device:Q_PNP_ECB
- added Q2, Q3: 2SC2021, symbol Device:Q_NPN_ECB
- added R1: 1M, symbol Device:R
- added R10: 220K, symbol Device:R
- added R11, R13: 1.2K, symbol Device:R
- added R12, R2: 510, symbol Device:R
- added R14, R15: 5.6K, symbol Device:R
- added R16: 10K, symbol Device:R
- added R17: 2.2K, symbol Device:R
- added R18, R19: 1K, symbol Device:R
- added R3, R4: 100, symbol Device:R
- added R5: 220, symbol Device:R
- added R6: 47K, symbol Device:R
- added R7, R9: 20K, symbol Device:R
- added R8: 12K, symbol Device:R
- added RA1: 12 x 10K, Resistor_THT:R_Array_SIP13, symbol Device:R_Network12
- added RA2: 4 x 6.8K, Resistor_THT:R_Array_SIP5, symbol Device:R_Network04
- added SW1: RESETSW, symbol Switch:SW_SPST
- added SW2: POWERSW, symbol Switch:SW_SPST
- added TC1: 30pF, symbol Device:C_Variable
- added U1: 6116 (WRAM), Package_DIP:DIP-24_W10.16mm, symbol NES-CPU-11:2KB_SRAM
- added U10: CIC, Package_DIP:DIP-16_W10.16mm, symbol NES-CPU-11:10NES_CIC
- added U2: 74HC373, Package_DIP:DIP-24_W10.16mm, symbol NES-CPU-11:74HC373
- added U3: 74HC139, Package_DIP:DIP-16_W7.62mm, symbol 74xx:74LS139
- added U4: 6116 (VRAM), Package_DIP:DIP-24_W10.16mm, symbol NES-CPU-11:2KB_SRAM
- added U5: RP2C02 PPU, Package_DIP:DIP-40_W15.24mm, symbol NES-CPU-11:RP2C02_PPU
- added U6: RP2A03 CPU, Package_DIP:DIP-40_W15.24mm, symbol NES-CPU-11:RP2A03_CPU
- added U7: 40H368 (CI), Package_DIP:DIP-16_W7.62mm, symbol NES-CPU-11:74HC368
- added U8: 40H368 (CII), Package_DIP:DIP-16_W7.62mm, symbol NES-CPU-11:74HC368
- added U9: 74LS04, Package_DIP:DIP-14_W7.62mm, symbol 74xx:74LS04
- added X1: 21.477272 MHz, symbol Device:Crystal_Small
- added X2: 4MHz, symbol Device:Crystal_Small
Connections:
- net labels added: +9V, 4016-D0, 4016-D1, 4016-D2, 4016-D3, 4016-D4, 4017-D0, 4017-D1, 4017-D2, 4017-D3, 4017-D4, AUDIO, CIC-CLK, CIC-RST, CIC-TO-CART, CIC-TO-MB, CPU-A0, CPU-A1, CPU-A10, CPU-A11, CPU-A12, CPU-A13, CPU-A14, CPU-A15, CPU-A2, CPU-A3, CPU-A4, CPU-A5, CPU-A6, CPU-A7, CPU-A8, CPU-A9, CPU-CLK, CPU-D0, CPU-D1, CPU-D2, CPU-D3, CPU-D4, CPU-D5, CPU-D6, CPU-D7, CPU-R~W, EXP-0, EXP-1, EXP-2, EXP-3, EXP-4, EXP-5, EXP-6, EXP-7, EXP-8, EXP-9, EXP-AUDIO-IN, EXP-AUDIO-OUT, EXP-VIDEO, OUT-0, OUT-1, OUT-2, PPU-A0, PPU-A1, PPU-A10, PPU-A11, PPU-A12, PPU-A13, PPU-A2, PPU-A3, PPU-A4, PPU-A5, PPU-A6, PPU-A7, PPU-A8, PPU-A9, PPU-CLK, PPU-D0, PPU-D1, PPU-D2, PPU-D3, PPU-D4, PPU-D5, PPU-D6, PPU-D7, PPU-D8, PPU-D9, PPU-~A13, PPU-~CE, PPU-~RD, PPU-~WE, SOUND-1, SOUND-2, SYSTEM-CLK, VCC, VIDEO, VRAM-A10, VRAM-~CE, WRAM-~CE, ~IRQ, ~NMI, ~OE1, ~OE2, ~ROMSEL, ~RST
- net labels removed: +5V, /CIC_CLK, /IRQ, /NMI, /OE1, /OE2, /RST, A0, A1, A10, A11, A12, A13, A14, A15, A2, A3, A4, A5, A6, A7, A8, A9, AUD1, AUD2, AUDIOIN, AUDIOOUT, BA0, BA1, BA10, BA11, BA12, BA2, BA3, BA4, BA5, BA6, BA7, BA8, BA9, BD0, BD1, BD2, BD3, BD4, BD5, BD6, BD7, CIC_2MB, CIC_2PAK, CIC_CLK, CIC_CLK0, CIC_CLK1, CIC_RST, CIC_RST0, CIC_RST1, CIC_SEED, CLK, D0, D1, D2, D3, D4, D5, D6, D7, EXP0, EXP1, EXP2, EXP3, EXP4, EXP5, EXP6, EXP7, EXP8, EXP9, JOY1/OE, JOY1D0, JOY1D1, JOY1D2, JOY1D3, JOY1D4, JOY2/OE, JOY2D0, JOY2D1, JOY2D2, JOY2D3, JOY2D4, OUT0, OUT1, OUT2, PRG-CE, R/W, SYS_CLK, U1-CE, U3A-G, U4-CE, U4-OE, U5-/A13, U5-/CS, U5-/R, U5-/W, U5-A13, U5-CLK, UNREG_VDD, VIDEOOUT, VOUT
- wire segments 478 -> 714
- no-connect marks 0 -> 8
Other:
- note added: "72-PIN CARTRIDGE CONNECTOR"
- note added: "CENTRAL PROCESSING UNIT & WORK RAM"
- note added: "CHECKING INTERGRATED CIRCUIT & POWER/RESET BOARD"
- note added: "CONTROLLER PORTS"
- note added: "CONTROLLER SHIFT REGISTERS"
- note added: "CPU, PPU, SYSTEM CLOCK CRYSTAL"
- note added: "EXPANSION CONNECTOR"
- note added: "FILTER CAPACITORS"
- note added: "MONO AUDIO MIXER & AMPLIFER"
- note added: "PICTURE PROCESSING UNIT & VIDEO RAM"

Commit message: Added .PDF and .kicad_pcb files
Parts:
- removed X2: 4MHz, symbol Device:Crystal_Small
- added R20: 100K, Capacitor_SMD:C_0603_1608Metric, symbol Device:R_Small
- added X2: 4MHz, Crystal:Resonator_muRata_CSTLSxxxG-3Pin_W8.0mm_H3.0mm, symbol Device:Crystal_GND2
- C11, C14, C17, C18: footprint (none) -> Capacitor_THT:C_Disc_D5.0mm_W2.5mm_P5.00mm
- C21: footprint (none) -> Capacitor_THT:C_Disc_D3.0mm_W1.6mm_P2.50mm
- C23, C9: footprint (none) -> Capacitor_THT:CP_Radial_D5.0mm_P2.50mm
- C4: footprint (none) -> Capacitor_THT:C_Disc_D5.0mm_W2.5mm_P2.50mm
- C6, C7: footprint (none) -> Capacitor_THT:C_Disc_D3.4mm_W2.1mm_P2.50mm
- C8: footprint (none) -> (none)
- D1, D2: footprint (none) -> Diode_THT:D_DO-35_SOD27_P10.16mm_Horizontal
- FC1: symbol Schematic:Ferrite_Core -> Motherboard-rescue:Ferrite_Core-Schematic
- FC2, R1, R10, R11, R12, R13, R14, R15, R16, R17, R18, R19, R2, R3, R4, R5, R6, R7, R8, R9: footprint (none) -> Resistor_THT:R_Axial_DIN0207_L6.3mm_D2.5mm_P10.16mm_Horizontal
- P1: footprint (none) -> NESRE:NES_Edge_Connector
- P2: footprint NesRE:NES_Edge_Connector -> NESRE:EXP_Header
- P3: footprint (none) -> NESRE:Mod_RF
- P6: footprint (none) -> NESRE:PowerReset-Switch-In
- TC1: footprint (none) -> NESRE:TrimmerCap-THT
- U1, U4: footprint Package_DIP:DIP-24_W10.16mm -> Package_DIP:DIP-24_W7.62mm
- U10: footprint Package_DIP:DIP-16_W10.16mm -> Package_DIP:DIP-16_W7.62mm
- U2: footprint Package_DIP:DIP-24_W10.16mm -> Package_DIP:DIP-20_W7.62mm
Connections:
- net labels removed: PPU-D8, PPU-D9
- wire segments 714 -> 710

Commit message: Finalized routing.
Parts:
- C4: footprint Capacitor_THT:C_Disc_D5.0mm_W2.5mm_P2.50mm -> Capacitor_THT:C_Disc_D5.0mm_W2.5mm_P5.00mm
- P3: symbol Connector:Conn_01x05_Male -> Connector:Conn_01x09_Male
- P4, P5: footprint (none) -> Connector_JST:JST_PH_S7B-PH-K_1x07_P2.00mm_Horizontal
Connections:
- wire segments 710 -> 713
Changed lines of the file:
@@
 Text Label 10750 2150 0    50   ~ 0
 GND
-Text Label 10750 1950 0    50   ~ 0
-CPU-A15
 Text Label 10750 1850 0    50   ~ 0
+CPU-A15
+Text Label 10750 1950 0    50   ~ 0
 M2
 Wire Wire Line
@@
 F 0 "P4" H 3350 1000 50  0000 C CNN
 F 1 "Controller Input" V 3550 1450 50  0000 C CNN
-F 2 "" H 3450 1450 50  0001 C CNN
+F 2 "Connector_JST:JST_PH_S7B-PH-K_1x07_P2.00mm_Horizontal" H 3450 1450 50  0001 C CNN
 F 3 "~" H 3450 1450 50  0001 C CNN
 	1    3450 1450
@@
 	4250 2300 4250 2000
 Wire Wire Line
-	3650 1150 4550 1150
-Wire Wire Line
 	3650 1350 4600 1350
 Wire Wire Line
@@
 	4100 1950 4100 1450
 Wire Wire Line
-	4400 950  4400 1950
-Wire Wire Line
 	4550 1150 4550 1950
 Wire Wire Line
@@
 	4550 1150 5700 1150
 Wire Wire Line
-	3650 1250 5500 1250
+	3650 1250 4400 1250
 Wire Wire Line
 	3950 1550 5100 1550
@@
 F 0 "P5" H 3350 2700 50  0000 C CNN
 F 1 "Controller Input" V 3550 3150 50  0000 C CNN
-F 2 "" H 3450 3150 50  0001 C CNN
+F 2 "Connector_JST:JST_PH_S7B-PH-K_1x07_P2.00mm_Horizontal" H 3450 3150 50  0001 C CNN
 F 3 "~" H 3450 3150 50  0001 C CNN
 	1    3450 3150
@@
 Wire Wire Line
 	4250 4000 4250 3700
-Wire Wire Line
-	3950 3650 3950 3350
-Wire Wire Line
-	4100 3650 4100 3250
-Wire Wire Line
-	4400 2650 4400 3150
-Wire Wire Line
-	3650 2950 4550 2950
 $Comp
 L Device:C_Small C31
@@
 Connection ~ 4900 3350
 Wire Wire Line
-	5100 3500 5100 3250
-Connection ~ 5100 3250
-Wire Wire Line
-	5300 3500 5300 3150
-Connection ~ 5300 3150
-Wire Wire Line
-	5500 3500 5500 2950
-Connection ~ 5500 2950
-Wire Wire Line
 	5700 3500 5700 2850
 Connection ~ 5700 2850
@@
 	5700 2850 6300 2850
 Wire Wire Line
-	5500 2950 6300 2950
-Wire Wire Line
-	5300 3150 6300 3150
-Wire Wire Line
 	5100 3250 6300 3250
 Wire Wire Line
@@
 	-1   0    0    1
 $EndComp
-Wire Wire Line
-	3650 2850 4700 2850
-Wire Wire Line
-	3650 3050 3900 3050
-Wire Wire Line
-	3650 3450 3800 3450
-Wire Wire Line
-	3650 3350 3950 3350
-Wire Wire Line
-	3800 2650 3800 3450
-Connection ~ 3800 3450
-Wire Wire Line
-	3800 3450 6300 3450
-Wire Wire Line
-	3900 3050 3900 3500
-Wire Wire Line
-	3900 3500 3800 3500
-Wire Wire Line
-	3800 3500 3800 3650
-Connection ~ 3900 3050
-Wire Wire Line
-	3900 3050 6300 3050
-Wire Wire Line
-	4550 3650 4550 2950
-Wire Wire Line
-	4700 2650 4700 2850
-Connection ~ 3950 3350
-Wire Wire Line
-	3950 3350 4900 3350
-Connection ~ 4100 3250
-Wire Wire Line
-	4100 3250 5100 3250
-Connection ~ 4400 3150
-Wire Wire Line
-	4400 3150 4400 3650
-Wire Wire Line
-	4400 3150 5300 3150
-Connection ~ 4550 2950
-Wire Wire Line
-	4550 2950 5500 2950
-Wire Wire Line
-	4550 2950 4550 2650
-Connection ~ 4700 2850
-Wire Wire Line
-	4700 2850 5700 2850
-Wire Wire Line
-	4700 2850 4700 3650
 $Comp
 L NES-CPU-11:74HC368 U7
@@
 	1    0    0    -1
 $EndComp
-Text Label 4450 5300 2    50   ~ 0
+Text Label 4200 5300 2    50   ~ 0
 AUDIO
 Text Label 4450 4750 2    50   ~ 0
@@
 L Device:C_Small C4
 U 1 1 5DD404CF
-P 3950 5750
-F 0 "C4" H 4150 5700 50  0000 C CNN
-F 1 "220pF" H 4150 5800 50  0000 C CNN
-F 2 "Capacitor_THT:C_Disc_D5.0mm_W2.5mm_P2.50mm" H 3950 5750 50  0001 C CNN
-F 3 "~" H 3950 5750 50  0001 C CNN
-	1    3950 5750
+P 3900 5400
+F 0 "C4" H 4100 5350 50  0000 C CNN
+F 1 "220pF" H 4100 5450 50  0000 C CNN
+F 2 "Capacitor_THT:C_Disc_D5.0mm_W2.5mm_P5.00mm" H 3900 5400 50  0001 C CNN
+F 3 "~" H 3900 5400 50  0001 C CNN
+	1    3900 5400
 	-1   0    0    1
 $EndComp
-Text Label 3950 6200 1    50   ~ 0
+Text Label 3900 5850 1    50   ~ 0
 GND
 Wire Wire Line
-	3950 5850 3950 6200
-Wire Wire Line
-	3950 5300 3950 5650
-Wire Wire Line
-	3900 5300 3950 5300
-Connection ~ 3950 5300
-Wire Wire Line
-	3950 5300 4450 5300
+	3900 5500 3900 5850
 Wire Wire Line
 	3500 4750 4450 4750
@@
 	8000 7700 7550 7700
 $Comp
-L Connector:Conn_01x05_Male P3
+L Connector:Conn_01x09_Male P3
 U 1 1 619A2E89
-P 8200 7000
-F 0 "P3" H 8172 6932 50  0000 R CNN
-F 1 "MOD RF" H 8172 7023 50  0000 R CNN
-F 2 "NESRE:Mod_RF" H 8200 7000 50  0001 C CNN
-F 3 "~" H 8200 7000 50  0001 C CNN
-	1    8200 7000
+P 8200 6800
+F 0 "P3" H 8172 6732 50  0000 R CNN
+F 1 "MOD RF" H 8172 6823 50  0000 R CNN
+F 2 "NESRE:Mod_RF" H 8200 6800 50  0001 C CNN
+F 3 "~" H 8200 6800 50  0001 C CNN
+	1    8200 6800
 	-1   0    0    1
 $EndComp
@@
 GND
 Text Label 7600 9300 3    50   ~ 0
-VCC
++9V
 $Comp
 L Device:C_Small C19
@@
 GND
 Text Label 11200 9300 3    50   ~ 0
-VCC
++9V
 $Comp
 L 74xx:74LS04 U9
 U 7 1 659B38AC
-P 7700 6250
-F 0 "U9" V 7333 6250 50  0000 C CNN
-F 1 "74LS04" V 7424 6250 50  0000 C CNN
-F 2 "Package_DIP:DIP-14_W7.62mm" H 7700 6250 50  0001 C CNN
-F 3 "http://www.ti.com/lit/gpn/sn74LS04" H 7700 6250 50  0001 C CNN
-	7    7700 6250
+P 7600 6150
+F 0 "U9" V 7233 6150 50  0000 C CNN
+F 1 "74LS04" V 7324 6150 50  0000 C CNN
+F 2 "Package_DIP:DIP-14_W7.62mm" H 7600 6150 50  0001 C CNN
+F 3 "http://www.ti.com/lit/gpn/sn74LS04" H 7600 6150 50  0001 C CNN
+	7    7600 6150
 	0    1    1    0
 $EndComp
 Wire Wire Line
-	7200 6250 6900 6250
+	7100 6150 6800 6150
 Wire Wire Line
-	8500 6250 8200 6250
-Text Label 6900 6250 0    50   ~ 0
+	8400 6150 8100 6150
+Text Label 6800 6150 0    50   ~ 0
 GND
-Text Label 8500 6250 2    50   ~ 0
+Text Label 8400 6150 2    50   ~ 0
 VCC
 Wire Wire Line
@@
 Text Label 5000 7150 1    50   ~ 0
 GND
+Connection ~ 3900 5300
+Wire Wire Line
+	3900 5300 4200 5300
+Text Label 8000 6400 2    50   ~ 0
+GND
+Text Label 8000 6500 2    50   ~ 0
+GND
+Text Label 8000 6600 2    50   ~ 0
+GND
+Text Label 8000 6700 2    50   ~ 0
+GND
+Wire Wire Line
+	5500 2950 6300 2950
+Connection ~ 5500 2950
+Wire Wire Line
+	5500 3500 5500 2950
+Wire Wire Line
+	5300 3150 6300 3150
+Connection ~ 5300 3150
+Wire Wire Line
+	5300 3500 5300 3150
+Wire Wire Line
+	5100 3500 5100 3250
+Connection ~ 5100 3250
+Wire Wire Line
+	3650 3050 3900 3050
+Wire Wire Line
+	3650 3450 3800 3450
+Wire Wire Line
+	3650 2850 4700 2850
+Wire Wire Line
+	3650 2950 4550 2950
+Wire Wire Line
+	3650 3150 4400 3150
+Wire Wire Line
+	3650 3250 4100 3250
+Wire Wire Line
+	3650 3350 3950 3350
+Wire Wire Line
+	3800 2650 3800 3450
+Connection ~ 3800 3450
+Wire Wire Line
+	3800 3450 6300 3450
+Wire Wire Line
+	3800 3650 3800 3500
+Wire Wire Line
+	3800 3500 3900 3500
+Wire Wire Line
+	3900 3500 3900 3050
+Connection ~ 3900 3050
+Wire Wire Line
+	3900 3050 6300 3050
+Wire Wire Line
+	3950 2650 3950 3350
+Connection ~ 3950 3350
+Wire Wire Line
+	3950 3350 4900 3350
+Wire Wire Line
+	3950 3350 3950 3650
+Wire Wire Line
+	4100 2650 4100 3250
+Connection ~ 4100 3250
+Wire Wire Line
+	4100 3250 5100 3250
+Wire Wire Line
+	4100 3250 4100 3650
+Wire Wire Line
+	4400 2650 4400 3150
+Connection ~ 4400 3150
+Wire Wire Line
+	4400 3150 5300 3150
+Wire Wire Line
+	4400 3150 4400 3650
+Wire Wire Line
+	4550 2650 4550 2950
+Connection ~ 4550 2950
+Wire Wire Line
+	4550 2950 5500 2950
+Wire Wire Line
+	4550 2950 4550 3650
+Wire Wire Line
+	4700 2650 4700 2850
+Connection ~ 4700 2850
+Wire Wire Line
+	4700 2850 5700 2850
+Wire Wire Line
+	4700 2850 4700 3650
+Wire Wire Line
+	4550 1150 4550 950
+Wire Wire Line
+	3650 1150 4550 1150
+Wire Wire Line
+	4400 950  4400 1250
+Connection ~ 4400 1250
 Wire Wire Line
-	4100 3250 3650 3250
+	4400 1250 5500 1250
 Wire Wire Line
-	4400 3150 3650 3150
+	4400 1250 4400 1950
 $EndSCHEMATC

Commit message: Completed board design
Parts:
- removed R20: 100K, Capacitor_SMD:C_0603_1608Metric, symbol Device:R_Small
- C20: footprint (none) -> Capacitor_THT:C_Disc_D3.0mm_W1.6mm_P2.50mm
- C41, C44, C5: footprint (none) -> Capacitor_THT:C_Disc_D3.0mm_W2.0mm_P2.50mm
- C42, C43, C45: footprint (none) -> Capacitor_THT:C_Disc_D3.4mm_W2.1mm_P2.50mm
- C8: footprint (none) -> Capacitor_THT:C_Disc_D7.0mm_W2.5mm_P5.00mm
- FC1: footprint (none) -> Resistor_THT:R_Axial_DIN0207_L6.3mm_D2.5mm_P10.16mm_Horizontal
- P6: footprint NESRE:PowerReset-Switch-In -> NESRE:PowerReset-switch-In
- Q1, Q2, Q3: footprint (none) -> Package_TO_SOT_THT:TO-126-3_Vertical
- R15: value 5.6K -> 100K
- X1: footprint (none) -> Crystal:Crystal_HC49-U_Horizontal_1EP_style2
Connections:
- wire segments 713 -> 714
Changed lines of the file:
@@
 F 0 "Q1" H 10741 8454 50  0000 L CNN
 F 1 "2SA937" H 10741 8545 50  0000 L CNN
-F 2 "" H 10750 8600 50  0001 C CNN
+F 2 "Package_TO_SOT_THT:TO-126-3_Vertical" H 10750 8600 50  0001 C CNN
 F 3 "~" H 10550 8500 50  0001 C CNN
 	1    10550 8500
@@
 F 0 "C5" H 11665 8496 50  0000 L CNN
 F 1 "330pF" H 11665 8405 50  0000 L CNN
-F 2 "" H 11588 8300 50  0001 C CNN
+F 2 "Capacitor_THT:C_Disc_D3.0mm_W2.0mm_P2.50mm" H 11588 8300 50  0001 C CNN
 F 3 "~" H 11550 8450 50  0001 C CNN
 	1    11550 8450
@@
 L Device:R R15
 U 1 1 60B446CF
-P 9000 3650
-F 0 "R15" V 8900 3450 50  0000 L CNN
-F 1 "5.6K" V 8900 3700 50  0000 L CNN
-F 2 "Resistor_THT:R_Axial_DIN0207_L6.3mm_D2.5mm_P10.16mm_Horizontal" V 8930 3650 50  0001 C CNN
-F 3 "~" H 9000 3650 50  0001 C CNN
-	1    9000 3650
+P 13150 6100
+F 0 "R15" V 13050 5900 50  0000 L CNN
+F 1 "100K" V 13050 6150 50  0000 L CNN
+F 2 "Resistor_THT:R_Axial_DIN0207_L6.3mm_D2.5mm_P10.16mm_Horizontal" V 13080 6100 50  0001 C CNN
+F 3 "~" H 13150 6100 50  0001 C CNN
+	1    13150 6100
 	1    0    0    -1
 $EndComp
-Text Label 9000 3250 3    50   ~ 0
-VCC
-Wire Wire Line
-	9000 3250 9000 3500
-Text Label 9000 4100 1    50   ~ 0
-~OE1
-Wire Wire Line
-	9000 4100 9000 3800
 $Comp
 L Device:C_Variable TC1
@@
 F 0 "C41" V 2829 7950 50  0000 C CNN
 F 1 "18pF" V 2738 7950 50  0000 C CNN
-F 2 "" H 2600 7950 50  0001 C CNN
+F 2 "Capacitor_THT:C_Disc_D3.0mm_W2.0mm_P2.50mm" H 2600 7950 50  0001 C CNN
 F 3 "~" H 2600 7950 50  0001 C CNN
 	1    2600 7950
@@
 F 0 "Q2" H 3240 7596 50  0000 L CNN
 F 1 "2SC2021" H 3240 7505 50  0000 L CNN
-F 2 "" H 3250 7650 50  0001 C CNN
+F 2 "Package_TO_SOT_THT:TO-126-3_Vertical" H 3250 7650 50  0001 C CNN
 F 3 "~" H 3050 7550 50  0001 C CNN
 	1    3050 7550
@@
 F 0 "Q3" H 1741 7596 50  0000 L CNN
 F 1 "2SC2021" H 1741 7505 50  0000 L CNN
-F 2 "" H 1750 7650 50  0001 C CNN
+F 2 "Package_TO_SOT_THT:TO-126-3_Vertical" H 1750 7650 50  0001 C CNN
 F 3 "~" H 1550 7550 50  0001 C CNN
 	1    1550 7550
@@
 F 0 "C42" H 1700 7750 50  0000 R CNN
 F 1 "15pF" H 1700 7850 50  0000 R CNN
-F 2 "" H 1850 7800 50  0001 C CNN
+F 2 "Capacitor_THT:C_Disc_D3.4mm_W2.1mm_P2.50mm" H 1850 7800 50  0001 C CNN
 F 3 "~" H 1850 7800 50  0001 C CNN
 	1    1850 7800
@@
 F 0 "C45" V 3779 8250 50  0000 C CNN
 F 1 "51pF" V 3688 8250 50  0000 C CNN
-F 2 "" H 3550 8250 50  0001 C CNN
+F 2 "Capacitor_THT:C_Disc_D3.4mm_W2.1mm_P2.50mm" H 3550 8250 50  0001 C CNN
 F 3 "~" H 3550 8250 50  0001 C CNN
 	1    3550 8250
 	0    -1   -1   0
 $EndComp
-Wire Wire Line
-	3300 8250 3450 8250
 $Comp
 L Device:C_Small C43
@@
 F 0 "C43" H 3050 8750 50  0000 C CNN
 F 1 "51pF" H 3050 8850 50  0000 C CNN
-F 2 "" H 2850 8800 50  0001 C CNN
+F 2 "Capacitor_THT:C_Disc_D3.4mm_W2.1mm_P2.50mm" H 2850 8800 50  0001 C CNN
 F 3 "~" H 2850 8800 50  0001 C CNN
 	1    2850 8800
@@
 F 0 "C44" V 1650 8550 50  0000 C CNN
 F 1 "220pF" V 1550 8550 50  0000 C CNN
-F 2 "" H 1800 8550 50  0001 C CNN
+F 2 "Capacitor_THT:C_Disc_D3.0mm_W2.0mm_P2.50mm" H 1800 8550 50  0001 C CNN
 F 3 "~" H 1800 8550 50  0001 C CNN
 	1    1800 8550
@@
 F 0 "X1" H 1900 8100 50  0000 C CNN
 F 1 "21.477272 MHz" H 2150 8000 50  0000 C CNN
-F 2 "" H 2100 7550 50  0001 C CNN
+F 2 "Crystal:Crystal_HC49-U_Horizontal_1EP_style2" H 2100 7550 50  0001 C CNN
 F 3 "~" H 2100 7550 50  0001 C CNN
 	1    2100 7550
@@
 F 0 "C20" V 3200 5050 50  0000 C CNN
 F 1 "51pF" V 3200 4850 50  0000 C CNN
-F 2 "" H 3100 4950 50  0001 C CNN
+F 2 "Capacitor_THT:C_Disc_D3.0mm_W1.6mm_P2.50mm" H 3100 4950 50  0001 C CNN
 F 3 "~" H 3100 4950 50  0001 C CNN
 	1    3100 4950
@@
 F 0 "FC1" H 3737 5125 50  0000 C CNN
 F 1 "39u" H 3737 5034 50  0000 C CNN
-F 2 "" H 3950 5100 50  0001 C CNN
+F 2 "Resistor_THT:R_Axial_DIN0207_L6.3mm_D2.5mm_P10.16mm_Horizontal" H 3950 5100 50  0001 C CNN
 F 3 "" H 3950 5100 50  0001 C CNN
 	1    3950 5100
@@
 F 0 "P6" H 8150 7500 50  0000 R CNN
 F 1 "PWR/RST IN" H 8150 7600 50  0000 R CNN
-F 2 "NESRE:PowerReset-Switch-In" H 8200 7600 50  0001 C CNN
+F 2 "NESRE:PowerReset-switch-In" H 8200 7600 50  0001 C CNN
 F 3 "~" H 8200 7600 50  0001 C CNN
 	1    8200 7600
@@
 F 0 "C8" V 6350 5600 50  0000 C CNN
 F 1 "100nF" V 6350 5400 50  0000 C CNN
-F 2 " " H 6250 5500 50  0001 C CNN
+F 2 "Capacitor_THT:C_Disc_D7.0mm_W2.5mm_P5.00mm" H 6250 5500 50  0001 C CNN
 F 3 "~" H 6250 5500 50  0001 C CNN
 	1    6250 5500
@@
 L 74xx:74LS04 U9
 U 7 1 659B38AC
-P 7600 6150
-F 0 "U9" V 7233 6150 50  0000 C CNN
-F 1 "74LS04" V 7324 6150 50  0000 C CNN
-F 2 "Package_DIP:DIP-14_W7.62mm" H 7600 6150 50  0001 C CNN
-F 3 "http://www.ti.com/lit/gpn/sn74LS04" H 7600 6150 50  0001 C CNN
-	7    7600 6150
+P 7600 6100
+F 0 "U9" V 7233 6100 50  0000 C CNN
+F 1 "74LS04" V 7324 6100 50  0000 C CNN
+F 2 "Package_DIP:DIP-14_W7.62mm" H 7600 6100 50  0001 C CNN
+F 3 "http://www.ti.com/lit/gpn/sn74LS04" H 7600 6100 50  0001 C CNN
+	7    7600 6100
 	0    1    1    0
 $EndComp
 Wire Wire Line
-	7100 6150 6800 6150
+	7100 6100 6800 6100
 Wire Wire Line
-	8400 6150 8100 6150
-Text Label 6800 6150 0    50   ~ 0
+	8400 6100 8100 6100
+Text Label 6800 6100 0    50   ~ 0
 GND
-Text Label 8400 6150 2    50   ~ 0
+Text Label 8400 6100 2    50   ~ 0
 VCC
 Wire Wire Line
@@
 	13150 6350 13950 6350
 Wire Wire Line
-	13150 6150 13150 6350
-Wire Wire Line
 	4850 6800 4850 7000
 $Comp
-L Device:R_Small R20
-U 1 1 5DB98916
-P 13150 6050
-F 0 "R20" H 13209 6096 50  0000 L CNN
-F 1 "100K" H 13209 6005 50  0000 L CNN
-F 2 "Capacitor_SMD:C_0603_1608Metric" H 13150 6050 50  0001 C CNN
-F 3 "~" H 13150 6050 50  0001 C CNN
-	1    13150 6050
-	1    0    0    -1
-$EndComp
-$Comp
 L Device:Crystal_GND2 X2
 U 1 1 5DB9934D
@@
 Wire Wire Line
 	4400 1250 4400 1950
+Wire Wire Line
+	3300 8250 3400 8250
+Wire Wire Line
+	3400 8250 3400 7200
+Wire Wire Line
+	3400 7200 3150 7200
+Connection ~ 3400 8250
+Wire Wire Line
+	3400 8250 3450 8250
+Wire Wire Line
+	13150 6250 13150 6350
 $EndSCHEMATC
