File: Board Files/Power Dual Mono Audio Comp Video/Motherboard.kicad_sch (KiCad schematic)
At the start: 17 parts, among them J3 , J4 Video, J5 R Audio, J6 L Audio, P6 MOD RF, Q4 BC817, U12 L7805

Commit message: Added board with built in AV/Power
Added board option with built in AV/Power and corrected the old oversized RCA place holders with accurate footprints.

Nothing is tested at this point but some quick eye math tells me that both boards can be combined.
Parts:
- J4, J5, J6: footprint Connector_Coaxial:BNC_Amphenol_B6252HB-NPP3G-50_Horizontal -> NESRE:RCA
Changed lines of the file:
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@@
       (effects (font (size 1.27 1.27)) (justify left))
     )
-    (property "Footprint" "Connector_Coaxial:BNC_Amphenol_B6252HB-NPP3G-50_Horizontal" (id 2) (at 231.14 109.22 0)
+    (property "Footprint" "NESRE:RCA" (id 2) (at 231.14 109.22 0)
       (effects (font (size 1.27 1.27)) hide)
     )
@@
       (effects (font (size 1.27 1.27)) (justify left))
     )
-    (property "Footprint" "Connector_Coaxial:BNC_Amphenol_B6252HB-NPP3G-50_Horizontal" (id 2) (at 231.14 118.11 0)
+    (property "Footprint" "NESRE:RCA" (id 2) (at 231.14 118.11 0)
       (effects (font (size 1.27 1.27)) hide)
     )
@@
       (effects (font (size 1.27 1.27)) (justify left))
     )
-    (property "Footprint" "Connector_Coaxial:BNC_Amphenol_B6252HB-NPP3G-50_Horizontal" (id 2) (at 219.71 118.11 0)
+    (property "Footprint" "NESRE:RCA" (id 2) (at 219.71 118.11 0)
       (effects (font (size 1.27 1.27)) hide)
     )
@@
     )
     (path "/6c57eb83-6e6a-40bc-a4f9-a1fc73ec9a6a"
-      (reference "J4") (unit 1) (value "Video") (footprint "Connector_Coaxial:BNC_Amphenol_B6252HB-NPP3G-50_Horizontal")
+      (reference "J4") (unit 1) (value "Video") (footprint "NESRE:RCA")
     )
     (path "/0b1d7959-5da3-4a8b-af77-fb6132d0ae4e"
-      (reference "J5") (unit 1) (value "R Audio") (footprint "Connector_Coaxial:BNC_Amphenol_B6252HB-NPP3G-50_Horizontal")
+      (reference "J5") (unit 1) (value "R Audio") (footprint "NESRE:RCA")
     )
     (path "/635813af-0a85-42f2-9a7d-f6500b4a91aa"
-      (reference "J6") (unit 1) (value "L Audio") (footprint "Connector_Coaxial:BNC_Amphenol_B6252HB-NPP3G-50_Horizontal")
+      (reference "J6") (unit 1) (value "L Audio") (footprint "NESRE:RCA")
     )
     (path "/ee3944ca-c505-472c-9b27-baea09596597"
